Commit message: update

File: ffw_description/gazebo/ffw_sh5_rev1_follower/ffw_sh5_follower.gazebo.xacro (robot description, xacro)
@@ -1,6 +1,5 @@
 <?xml version="1.0"?>
 <robot xmlns:xacro="http://ros.org/wiki/xacro">
-  <!-- prefix is optional; default empty for non-prefixed TF/frames -->
-  <xacro:macro name="ffw_sg2_follower_gazebo" params="prefix:=">
+<xacro:macro name="ffw_sh5_follower_gazebo" params="prefix:=''">
   <xacro:macro name="SimpleTransmission" params="trans joint actuator">
     <transmission name="${trans}">
@@ -43,14 +42,4 @@
   <xacro:Link reference="arm_l_link6"/>
   <xacro:Link reference="arm_l_link7"/>
-  <xacro:Link reference="r_rh_p12_rn_base"/>
-  <xacro:Link reference="r_rh_p12_rn_r1"/>
-  <xacro:Link reference="r_rh_p12_rn_r2"/>
-  <xacro:Link reference="r_rh_p12_rn_l1"/>
-  <xacro:Link reference="r_rh_p12_rn_l2"/>
-  <xacro:Link reference="l_rh_p12_rn_base"/>
-  <xacro:Link reference="l_rh_p12_rn_r1"/>
-  <xacro:Link reference="l_rh_p12_rn_r2"/>
-  <xacro:Link reference="l_rh_p12_rn_l1"/>
-  <xacro:Link reference="l_rh_p12_rn_l2"/>
   <xacro:SimpleTransmission trans="lift_trans" joint="lift_joint" actuator="lift_actuator"/>
   <xacro:SimpleTransmission trans="head_trans1" joint="head_joint1" actuator="head_actuator1"/>
@@ -70,13 +59,44 @@
   <xacro:SimpleTransmission trans="arm_l_trans6" joint="arm_l_joint6" actuator="arm_l_actuator6"/>
   <xacro:SimpleTransmission trans="arm_l_trans7" joint="arm_l_joint7" actuator="arm_l_actuator7"/>
-  <xacro:SimpleTransmission trans="r_tran_r1" joint="r_rh_r1_joint" actuator="r_actuator1" />
-  <xacro:SimpleTransmission trans="r_tran_r2" joint="r_rh_r2" actuator="r_actuator2" />
-  <xacro:SimpleTransmission trans="r_tran_l1" joint="r_rh_l1" actuator="r_actuator3" />
-  <xacro:SimpleTransmission trans="r_tran_l2" joint="r_rh_l2" actuator="r_actuator4" />
-  <xacro:SimpleTransmission trans="l_tran_r1" joint="l_rh_r1_joint" actuator="l_actuator1" />
-  <xacro:SimpleTransmission trans="l_tran_r2" joint="l_rh_r2" actuator="l_actuator2" />
-  <xacro:SimpleTransmission trans="l_tran_l1" joint="l_rh_l1" actuator="l_actuator3" />
-  <xacro:SimpleTransmission trans="l_tran_l2" joint="l_rh_l2" actuator="l_actuator4" />
-  <!-- GZ lidar sensors for simulation (publish Gazebo LaserScan; bridge to ROS if needed) -->
+  <xacro:SimpleTransmission trans="hand_l_trans1" joint="finger_l_joint1" actuator="hand_l_actuator1"/>
+  <xacro:SimpleTransmission trans="hand_l_trans2" joint="finger_l_joint2" actuator="hand_l_actuator2"/>
+  <xacro:SimpleTransmission trans="hand_l_trans3" joint="finger_l_joint3" actuator="hand_l_actuator3"/>
+  <xacro:SimpleTransmission trans="hand_l_trans4" joint="finger_l_joint4" actuator="hand_l_actuator4"/>
+  <xacro:SimpleTransmission trans="hand_l_trans5" joint="finger_l_joint5" actuator="hand_l_actuator5"/>
+  <xacro:SimpleTransmission trans="hand_l_trans6" joint="finger_l_joint6" actuator="hand_l_actuator6"/>
+  <xacro:SimpleTransmission trans="hand_l_trans7" joint="finger_l_joint7" actuator="hand_l_actuator7"/>
+  <xacro:SimpleTransmission trans="hand_l_trans8" joint="finger_l_joint8" actuator="hand_l_actuator8"/>
+  <xacro:SimpleTransmission trans="hand_l_trans9" joint="finger_l_joint9" actuator="hand_l_actuator9"/>
+  <xacro:SimpleTransmission trans="hand_l_trans10" joint="finger_l_joint10" actuator="hand_l_actuator10"/>
+  <xacro:SimpleTransmission trans="hand_l_trans11" joint="finger_l_joint11" actuator="hand_l_actuator11"/>
+  <xacro:SimpleTransmission trans="hand_l_trans12" joint="finger_l_joint12" actuator="hand_l_actuator12"/>
+  <xacro:SimpleTransmission trans="hand_l_trans13" joint="finger_l_joint13" actuator="hand_l_actuator13"/>
+  <xacro:SimpleTransmission trans="hand_l_trans14" joint="finger_l_joint14" actuator="hand_l_actuator14"/>
+  <xacro:SimpleTransmission trans="hand_l_trans15" joint="finger_l_joint15" actuator="hand_l_actuator15"/>
+  <xacro:SimpleTransmission trans="hand_l_trans16" joint="finger_l_joint16" actuator="hand_l_actuator16"/>
+  <xacro:SimpleTransmission trans="hand_l_trans17" joint="finger_l_joint17" actuator="hand_l_actuator17"/>
+  <xacro:SimpleTransmission trans="hand_l_trans18" joint="finger_l_joint18" actuator="hand_l_actuator18"/>
+  <xacro:SimpleTransmission trans="hand_l_trans19" joint="finger_l_joint19" actuator="hand_l_actuator19"/>
+  <xacro:SimpleTransmission trans="hand_l_trans20" joint="finger_l_joint20" actuator="hand_l_actuator20"/>
+  <xacro:SimpleTransmission trans="hand_r_trans1" joint="finger_r_joint1" actuator="hand_r_actuator1"/>
+  <xacro:SimpleTransmission trans="hand_r_trans2" joint="finger_r_joint2" actuator="hand_r_actuator2"/>
+  <xacro:SimpleTransmission trans="hand_r_trans3" joint="finger_r_joint3" actuator="hand_r_actuator3"/>
+  <xacro:SimpleTransmission trans="hand_r_trans4" joint="finger_r_joint4" actuator="hand_r_actuator4"/>
+  <xacro:SimpleTransmission trans="hand_r_trans5" joint="finger_r_joint5" actuator="hand_r_actuator5"/>
+  <xacro:SimpleTransmission trans="hand_r_trans6" joint="finger_r_joint6" actuator="hand_r_actuator6"/>
+  <xacro:SimpleTransmission trans="hand_r_trans7" joint="finger_r_joint7" actuator="hand_r_actuator7"/>
+  <xacro:SimpleTransmission trans="hand_r_trans8" joint="finger_r_joint8" actuator="hand_r_actuator8"/>
+  <xacro:SimpleTransmission trans="hand_r_trans9" joint="finger_r_joint9" actuator="hand_r_actuator9"/>
+  <xacro:SimpleTransmission trans="hand_r_trans10" joint="finger_r_joint10" actuator="hand_r_actuator10"/>
+  <xacro:SimpleTransmission trans="hand_r_trans11" joint="finger_r_joint11" actuator="hand_r_actuator11"/>
+  <xacro:SimpleTransmission trans="hand_r_trans12" joint="finger_r_joint12" actuator="hand_r_actuator12"/>
+  <xacro:SimpleTransmission trans="hand_r_trans13" joint="finger_r_joint13" actuator="hand_r_actuator13"/>
+  <xacro:SimpleTransmission trans="hand_r_trans14" joint="finger_r_joint14" actuator="hand_r_actuator14"/>
+  <xacro:SimpleTransmission trans="hand_r_trans15" joint="finger_r_joint15" actuator="hand_r_actuator15"/>
+  <xacro:SimpleTransmission trans="hand_r_trans16" joint="finger_r_joint16" actuator="hand_r_actuator16"/>
+  <xacro:SimpleTransmission trans="hand_r_trans17" joint="finger_r_joint17" actuator="hand_r_actuator17"/>
+  <xacro:SimpleTransmission trans="hand_r_trans18" joint="finger_r_joint18" actuator="hand_r_actuator18"/>
+  <xacro:SimpleTransmission trans="hand_r_trans19" joint="finger_r_joint19" actuator="hand_r_actuator19"/>
+  <xacro:SimpleTransmission trans="hand_r_trans20" joint="finger_r_joint20" actuator="hand_r_actuator20"/>
   <gazebo reference="lidar_l_link">
     <sensor name="lidar_left" type="gpu_lidar">

File: ffw_description/ros2_control/ffw_sh5_rev1_follower/ffw_sh5_sensor.ros2_control.xacro (robot description, xacro)
@@ -1,6 +1,6 @@
 <?xml version="1.0"?>
 <robot xmlns:xacro="http://www.ros.org/wiki/xacro">
-  <xacro:macro name="ffw_sg2_sensor_system" params="use_sim:=^|false use_mock_hardware:=^|false mock_sensor_commands:=^|false">
-    <ros2_control name="ffw_sg2_sensor" type="system" is_async="true">
+  <xacro:macro name="ffw_sh5_sensor_system" params="use_sim:=^|false use_mock_hardware:=^|false mock_sensor_commands:=^|false">
+    <ros2_control name="ffw_sh5_sensor" type="system" is_async="true">
       <xacro:unless value="$(arg use_sim)">
         <hardware>

File: ffw_description/urdf/ffw_sh5_rev1_follower/ffw_sh5_follower.urdf.xacro (robot description, xacro)
@@ -1,18 +1,19 @@
 <?xml version="1.0"?>
-<robot xmlns:xacro="http://www.ros.org/wiki/xacro" name="ffw_sg2_follower">
+<robot xmlns:xacro="http://www.ros.org/wiki/xacro" name="ffw_sh5_follower">
   <xacro:property name="meshes_file_direction" value="package://ffw_description/meshes/$(arg model)" />
   <xacro:property name="swerve_meshes_dir" value="package://ffw_description/meshes/common/follower/swerve" />
-  <xacro:arg name="use_sim" default="false" />
+  <xacro:arg name="use_sim" default="true" />
   <xacro:arg name="use_mock_hardware" default="false" />
   <xacro:arg name="mock_sensor_commands" default="false" />
   <xacro:arg name="prefix" default="" />
-  <xacro:arg name="model" default="ffw_sg2_rev1_follower" />
-  <xacro:arg name="ros2_control_type" default="ffw_sg2_follower" />
+  <xacro:arg name="model" default="ffw_sh5_rev1_follower" />
   <xacro:include filename="$(find ffw_description)/urdf/common/follower/ffw_follower_body.xacro" />
-  <xacro:include filename="$(find ffw_description)/urdf/common/rh_p12_rn_a/rh_p12_rn_a.urdf.xacro" />
-  <xacro:include filename="$(find ffw_description)/ros2_control/$(arg model)/$(arg ros2_control_type).ros2_control.xacro" />
-  <xacro:include filename="$(find ffw_description)/ros2_control/$(arg model)/ffw_sg2_base.ros2_control.xacro" />
-  <xacro:include filename="$(find ffw_description)/ros2_control/$(arg model)/ffw_sg2_sensor.ros2_control.xacro" />
-  <xacro:include filename="$(find ffw_description)/gazebo/$(arg model)/ffw_sg2_follower.gazebo.xacro" />
+  <xacro:include filename="$(find ffw_description)/urdf/common/hx5_d20/hx5_d20_left.urdf.xacro" />
+  <xacro:include filename="$(find ffw_description)/urdf/common/hx5_d20/hx5_d20_right.urdf.xacro" />
+  <xacro:include filename="$(find ffw_description)/ros2_control/$(arg model)/ffw_sh5_follower.ros2_control.xacro" />
+  <xacro:include filename="$(find ffw_description)/ros2_control/$(arg model)/ffw_sh5_base.ros2_control.xacro" />
+  <xacro:include filename="$(find ffw_description)/ros2_control/$(arg model)/ffw_sh5_sensor.ros2_control.xacro" />
+  <xacro:include filename="$(find ffw_description)/gazebo/$(arg model)/ffw_sh5_follower.gazebo.xacro" />
+  <xacro:ffw_sh5_follower_gazebo prefix="$(arg prefix)" />
   <link name="$(arg prefix)base_link">
     <visual>
@@ -56,5 +57,5 @@
       <material name="black"><color rgba="0.1 0.1 0.1 1"/></material>
     </visual>
-  </link>
+      </link>
   <joint name="$(arg prefix)lidar_r_joint" type="fixed">
     <parent link="$(arg prefix)base_link"/>
@@ -62,6 +63,17 @@
     <origin xyz="-0.111881 -0.240 0.34432" rpy="0 0 -1.57079632679"/>
   </joint>
-  <!-- <link name="$(arg prefix)lidar_r_link">
-  </link> -->
+  <link name="$(arg prefix)lidar_r_link">
+    <inertial>
+      <mass value="0.1"/>
+      <origin xyz="0 0 0" rpy="0 0 0"/>
+      <inertia ixx="0.0001" ixy="0" ixz="0" iyy="0.0001" iyz="0" izz="0.0001"/>
+    </inertial>
+    <visual>
+      <geometry>
+        <cylinder radius="0.03" length="0.03"/>
+      </geometry>
+      <material name="black"><color rgba="0.1 0.1 0.1 1"/></material>
+    </visual>
+  </link>
   <joint name="$(arg prefix)imu_joint" type="fixed">
     <parent link="$(arg prefix)base_link"/>
@@ -70,17 +82,4 @@
   </joint>
   <link name="$(arg prefix)imu_link">
-  </link>
-  <link name="$(arg prefix)lidar_r_link">
-    <inertial>
-      <mass value="0.1"/>
-      <origin xyz="0 0 0" rpy="0 0 0"/>
-      <inertia ixx="0.0001" ixy="0" ixz="0" iyy="0.0001" iyz="0" izz="0.0001"/>
-    </inertial>
-    <visual>
-      <geometry>
-        <cylinder radius="0.03" length="0.03"/>
-      </geometry>
-      <material name="black"><color rgba="0.1 0.1 0.1 1"/></material>
-    </visual>
   </link>
   <link name="$(arg prefix)lift_link">
@@ -113,47 +112,13 @@
     <origin xyz="0.0 0.0 0.0" rpy="0 0 0"/>
   </joint>
-  <!-- Gazebo plugins/sensors -->
-  <xacro:ffw_sg2_follower_gazebo prefix="$(arg prefix)" />
   <xacro:ffw_follower_body parent="$(arg prefix)base_link" prefix="$(arg prefix)">
     <origin xyz="-0.0199 0 1.4316" rpy="0 0 0" />
   </xacro:ffw_follower_body>
-  <xacro:rh_p12_rn_a parent="$(arg prefix)arm_l_link7" prefix="$(arg prefix)gripper_l_">
-    <origin xyz="0 0 -0.078" rpy="0 3.14159265359 3.14159265359"/>
-  </xacro:rh_p12_rn_a>
-  <joint name="$(arg prefix)end_effector_l_joint" type="fixed">
-    <parent link="$(arg prefix)arm_l_link7"/>
-    <child link="$(arg prefix)end_effector_l_link"/>
-    <origin xyz="0 0 -0.215" rpy="0 0 0"/>
-  </joint>
-  <link name="$(arg prefix)end_effector_l_link">
-    <visual>
-      <origin xyz="0 0 0" rpy="0 0 0"/>
-      <geometry>
-        <box size="0.01 0.01 0.01" />
-      </geometry>
-      <material name="red">
-        <color rgba="1.0 0.0 0.0 1"/>
-      </material>
-    </visual>
-  </link>
-  <xacro:rh_p12_rn_a parent="$(arg prefix)arm_r_link7" prefix="$(arg prefix)gripper_r_">
-    <origin xyz="0 0 -0.078" rpy="0 3.14159265359 3.14159265359"/>
-  </xacro:rh_p12_rn_a>
-  <joint name="$(arg prefix)end_effector_r_joint" type="fixed">
-    <parent link="$(arg prefix)arm_r_link7"/>
-    <child link="$(arg prefix)end_effector_r_link"/>
-    <origin xyz="0 0 -0.215" rpy="0 0 0"/>
-  </joint>
-  <link name="$(arg prefix)end_effector_r_link">
-    <visual>
-      <origin xyz="0 0 0" rpy="0 0 0"/>
-      <geometry>
-        <box size="0.01 0.01 0.01" />
-      </geometry>
-      <material name="red">
-        <color rgba="1.0 0.0 0.0 1"/>
-      </material>
-    </visual>
-  </link>
+  <xacro:hx5_d20_left parent="$(arg prefix)arm_l_link7" prefix="$(arg prefix)">
+    <origin xyz="0 0 -0.078" rpy="0 3.14159265359 1.5708"/>
+  </xacro:hx5_d20_left>
+  <xacro:hx5_d20_right parent="$(arg prefix)arm_r_link7" prefix="$(arg prefix)">
+    <origin xyz="0 0 -0.078" rpy="0 3.14159265359 -1.5708"/>
+  </xacro:hx5_d20_right>
   <joint name="$(arg prefix)left_wheel_steer" type="revolute">
       <parent link="$(arg prefix)base_link"/>
@@ -200,6 +165,6 @@
         <mesh filename="${swerve_meshes_dir}/left_wheel_drive_link.stl" scale="0.001 0.001 0.001" />
       </geometry>
-      <material name="black">
-        <color rgba="0.1 0.1 0.1 1.0"/>
+      <material name="silver">
+        <color rgba="0.75 0.75 0.75 1"/>
       </material>
     </visual>
@@ -268,6 +233,6 @@
         <mesh filename="${swerve_meshes_dir}/right_wheel_drive_link.stl" scale="0.001 0.001 0.001" />
       </geometry>
-      <material name="black">
-        <color rgba="0.1 0.1 0.1 1.0"/>
+      <material name="silver">
+        <color rgba="0.75 0.75 0.75 1"/>
       </material>
     </visual>
@@ -340,4 +305,10 @@
       </material>
     </visual>
+    <!-- <collision>
+      <origin xyz="0 0 0" rpy="0 0 0" />
+      <geometry>
+        <mesh filename="${swerve_meshes_dir}/rear_wheel_drive_link.stl" scale="0.001 0.001 0.001" />
+      </geometry>
+    </collision> -->
     <collision>
       <origin xyz="0 0 0" rpy="1.5708 0 0"/>
@@ -346,10 +317,4 @@
       </geometry>
     </collision>
-    <!-- <collision>
-      <origin xyz="0 0 0" rpy="0 0 0" />
-      <geometry>
-        <mesh filename="${swerve_meshes_dir}/rear_wheel_drive_link.stl" scale="0.001 0.001 0.001" />
-      </geometry>
-    </collision> -->
     <inertial>
        <origin xyz="0.000000000e+00 1.499601700e-03 0.000000000e+00" />
@@ -360,13 +325,13 @@
     </inertial>
   </link>
-  <xacro:ffw_sg2_follower_system
+  <xacro:ffw_sh5_follower_system
     use_sim="$(arg use_sim)"
     use_mock_hardware="$(arg use_mock_hardware)"
     mock_sensor_commands="$(arg mock_sensor_commands)"/>
-  <xacro:ffw_sg2_base_system
+  <xacro:ffw_sh5_base_system
     use_sim="$(arg use_sim)"
     use_mock_hardware="$(arg use_mock_hardware)"
     mock_sensor_commands="$(arg mock_sensor_commands)"/>
-  <xacro:ffw_sg2_sensor_system
+  <xacro:ffw_sh5_sensor_system
     use_sim="$(arg use_sim)"
     use_mock_hardware="$(arg use_mock_hardware)"
@@ -374,5 +339,5 @@
   <gazebo>
       <plugin filename="gz_ros2_control-system" name="gz_ros2_control::GazeboSimROS2ControlPlugin">
-        <parameters>$(find ffw_bringup)/config/$(arg model)/ffw_sg2_follower_ai_hardware_controller.yaml</parameters>
+        <parameters>$(find ffw_bringup)/config/$(arg model)/ffw_sh5_follower_ai_hardware_controller.yaml</parameters>
       </plugin>
   </gazebo>
