Commit message: update

File: ffw_description/gazebo/ffw_sh5_rev1_follower/ffw_sh5_follower.gazebo.xacro (robot description, xacro)
@@ -17,4 +17,5 @@
     <gazebo reference="${reference}">
       <kp>1000000.0</kp>
+      <!-- <gravity>false</gravity> -->
       <kd>100.0</kd>
       <mu1>30.0</mu1>
@@ -160,5 +161,5 @@
   </gazebo>
   <!-- RealSense D405 Left Camera (on arm_l_link7) -->
-  <!-- <gazebo reference="camera_l_link">
+  <gazebo reference="camera_l_link">
     <sensor name="camera_l_rgb" type="camera">
       <always_on>true</always_on>
@@ -189,5 +190,5 @@
       <update_rate>30.0</update_rate>
       <visualize>false</visualize>
-      <topic>camera_l/depth</topic>
+      <topic>camera_l</topic>
       <gz_frame_id>camera_l_link</gz_frame_id>
       <camera>
@@ -203,7 +204,7 @@
       </camera>
     </sensor>
-  </gazebo> -->
+  </gazebo>
   <!-- RealSense D405 Right Camera (on arm_r_link7) -->
-  <!-- <gazebo reference="camera_r_link">
+  <gazebo reference="camera_r_link">
     <sensor name="camera_r_rgb" type="camera">
       <always_on>true</always_on>
@@ -234,5 +235,5 @@
       <update_rate>30.0</update_rate>
       <visualize>false</visualize>
-      <topic>camera_r/depth</topic>
+      <topic>camera_r</topic>
       <gz_frame_id>camera_r_link</gz_frame_id>
       <camera>
@@ -248,7 +249,7 @@
       </camera>
     </sensor>
-  </gazebo> -->
+  </gazebo>
  <!-- ZED Mini Camera (single RGB) -->
-  <!-- <gazebo reference="zedm_camera_center">
+  <gazebo reference="zedm_camera_center">
     <sensor name="zedm" type="camera">
       <always_on>true</always_on>
@@ -270,5 +271,30 @@
       </camera>
     </sensor>
-  </gazebo> -->
+  <sensor name="zedm_rgbd" type="rgbd_camera">
+    <always_on>true</always_on>
+    <update_rate>15.0</update_rate>
+    <topic>zedm</topic>
+    <gz_frame_id>zedm_camera_center</gz_frame_id>
+    <camera>
+      <horizontal_fov>1.7453293</horizontal_fov>
+      <image>
+        <width>640</width>
+        <height>360</height>
+        <format>R8G8B8</format>
+      </image>
+      <clip><near>0.3</near><far>10.0</far></clip>
+      <depth_camera>
+        <output>depths</output>
+        <clip><near>0.3</near><far>10.0</far></clip>
+      </depth_camera>
+      <lens>
+        <intrinsics>
+          <fx>525</fx><fy>525</fy>
+          <cx>320</cx><cy>180</cy>
+        </intrinsics>
+      </lens>
+    </camera>
+  </sensor>
+  </gazebo>
   </xacro:macro>
 </robot>

File: ffw_description/ros2_control/ffw_sh5_rev1_follower/ffw_sh5_base.ros2_control.xacro (robot description, xacro)
@@ -2,5 +2,5 @@
 <robot xmlns:xacro="http://www.ros.org/wiki/xacro">
   <xacro:macro name="ffw_sh5_base_system" params="use_sim:=^|false use_mock_hardware:=^|false mock_sensor_commands:=^|false">
-    <ros2_control name="ffw_sh5_base" type="system" is_async="true">
+    <ros2_control name="ffw_sh5_base" type="system" is_async="false">
       <xacro:if value="$(arg use_sim)">
         <hardware>

File: ffw_description/ros2_control/ffw_sh5_rev1_follower/ffw_sh5_follower.ros2_control.xacro (robot description, xacro)
@@ -2,5 +2,5 @@
 <robot xmlns:xacro="http://www.ros.org/wiki/xacro">
   <xacro:macro name="ffw_sh5_follower_system" params="use_sim:=^|false use_mock_hardware:=^|false mock_sensor_commands:=^|false">
-    <ros2_control name="ffw_sh5_follower" type="system" is_async="true">
+    <ros2_control name="ffw_sh5_follower" type="system" is_async="false">
       <xacro:if value="$(arg use_sim)">
         <hardware>

File: ffw_description/ros2_control/ffw_sh5_rev1_follower/ffw_sh5_sensor.ros2_control.xacro (robot description, xacro)
@@ -2,5 +2,5 @@
 <robot xmlns:xacro="http://www.ros.org/wiki/xacro">
   <xacro:macro name="ffw_sh5_sensor_system" params="use_sim:=^|false use_mock_hardware:=^|false mock_sensor_commands:=^|false">
-    <ros2_control name="ffw_sh5_sensor" type="system" is_async="true">
+    <ros2_control name="ffw_sh5_sensor" type="system" is_async="false">
       <xacro:unless value="$(arg use_sim)">
         <hardware>

File: ffw_description/urdf/common/follower/ffw_follower_body.xacro (robot description, xacro)
@@ -103,5 +103,5 @@
       <xacro:zed_camera name="zedm" model="zedm" />
       <joint name="zedm_joint" type="fixed">
-         <parent link="head_link2"/>
+         <parent link="${prefix}head_link2"/>
          <child link="zedm_camera_link"/>
          <origin xyz="0.0238122 -0.00651797 -0.0242094" rpy="0 0 0" />
@@ -112,5 +112,5 @@
          <origin xyz="0 0.1045 0" rpy="0 0 0" />
          <axis xyz="0 1 0" />
-         <limit velocity="4.8" effort="1000" lower="-3.14" upper="3.14" />
+         <limit velocity="4.8" effort="1000" lower="-3.15" upper="3.15" />
          <dynamics damping="0.1" />
       </joint>
@@ -144,5 +144,5 @@
          <origin xyz="0 0.123 0" rpy="0 0 0" />
          <axis xyz="1 0 0" />
-         <limit velocity="4.8" effort="1000" lower="0.0" upper="3.14" />
+         <limit velocity="4.8" effort="1000" lower="-3.14" upper="3.14" />
          <dynamics damping="0.1" />
       </joint>
@@ -176,5 +176,5 @@
          <origin xyz="0 0 -0.165" rpy="0 0 0" />
          <axis xyz="0 0 1" />
-         <limit velocity="4.8" effort="1000" lower="-3.14" upper="3.14" />
+         <limit velocity="4.8" effort="1000" lower="-3.15" upper="3.15" />
          <dynamics damping="0.1" />
       </joint>
@@ -240,5 +240,5 @@
          <origin xyz="-0.041004 0 -0.1489" rpy="0 0 0" />
          <axis xyz="0 0 1" />
-         <limit velocity="4.8" effort="1000" lower="-3.14" upper="3.14" />
+         <limit velocity="4.8" effort="1000" lower="-3.15" upper="3.15" />
          <dynamics damping="0.1" />
       </joint>
@@ -304,5 +304,5 @@
          <origin xyz="0 0 -0.0885" rpy="0 0 0" />
          <axis xyz="1 0 0" />
-         <limit velocity="4.8" effort="1000" lower="-1.8201" upper="1.5804" />
+         <limit velocity="4.8" effort="1000" lower="-1.85" upper="1.6" />
          <dynamics damping="0.1" />
       </joint>
@@ -339,5 +339,5 @@
          <origin xyz="0 -0.1045 0" rpy="0 0 0" />
          <axis xyz="0 1 0" />
-         <limit velocity="4.8" effort="1000" lower="-3.14" upper="3.14" />
+         <limit velocity="4.8" effort="1000" lower="-3.15" upper="3.15" />
          <dynamics damping="0.1" />
       </joint>
@@ -371,5 +371,5 @@
          <origin xyz="0 -0.123 0" rpy="0 0 0" />
          <axis xyz="1 0 0" />
-         <limit velocity="4.8" effort="1000" lower="-3.14" upper="0" />
+         <limit velocity="4.8" effort="1000" lower="-3.14" upper="3.14" />
          <dynamics damping="0.1" />
       </joint>
@@ -467,5 +467,5 @@
          <origin xyz="-0.041004 0 -0.1489" rpy="0 0 0" />
          <axis xyz="0 0 1" />
-         <limit velocity="4.8" effort="1000" lower="-3.14" upper="3.14" />
+         <limit velocity="4.8" effort="1000" lower="-3.15" upper="3.15" />
          <dynamics damping="0.1" />
       </joint>
@@ -531,5 +531,5 @@
          <origin xyz="0 0 -0.0885" rpy="0 0 0" />
          <axis xyz="1 0 0" />
-         <limit velocity="4.8" effort="1000" lower="-1.5804" upper="1.8201" />
+         <limit velocity="4.8" effort="1000" lower="-1.59" upper="1.83" />
          <dynamics damping="0.1" />
       </joint>

File: ffw_description/urdf/ffw_sh5_rev1_follower/ffw_sh5_follower.urdf.xacro (robot description, xacro)
@@ -134,6 +134,6 @@
         <mesh filename="${swerve_meshes_dir}/left_wheel_steer_link.stl" scale="0.001 0.001 0.001" />
       </geometry>
-      <material name="silver">
-        <color rgba="0.75 0.75 0.75 1"/>
+      <material name="black">
+        <color rgba="0.1 0.1 0.1 1"/>
       </material>
     </visual>
@@ -165,6 +165,6 @@
         <mesh filename="${swerve_meshes_dir}/left_wheel_drive_link.stl" scale="0.001 0.001 0.001" />
       </geometry>
-      <material name="silver">
-        <color rgba="0.75 0.75 0.75 1"/>
+      <material name="black">
+        <color rgba="0.1 0.1 0.1 1"/>
       </material>
     </visual>
@@ -202,6 +202,6 @@
         <mesh filename="${swerve_meshes_dir}/right_wheel_steer_link.stl" scale="0.001 0.001 0.001" />
       </geometry>
-      <material name="silver">
-        <color rgba="0.75 0.75 0.75 1"/>
+      <material name="black">
+        <color rgba="0.1 0.1 0.1 1"/>
       </material>
     </visual>
@@ -233,6 +233,6 @@
         <mesh filename="${swerve_meshes_dir}/right_wheel_drive_link.stl" scale="0.001 0.001 0.001" />
       </geometry>
-      <material name="silver">
-        <color rgba="0.75 0.75 0.75 1"/>
+      <material name="black">
+        <color rgba="0.1 0.1 0.1 1"/>
       </material>
     </visual>
@@ -270,6 +270,6 @@
         <mesh filename="${swerve_meshes_dir}/rear_wheel_steer_link.stl" scale="0.001 0.001 0.001" />
       </geometry>
-      <material name="silver">
-        <color rgba="0.75 0.75 0.75 1"/>
+      <material name="black">
+        <color rgba="0.1 0.1 0.1 1"/>
       </material>
     </visual>
@@ -301,6 +301,6 @@
         <mesh filename="${swerve_meshes_dir}/rear_wheel_drive_link.stl" scale="0.001 0.001 0.001" />
       </geometry>
-      <material name="silver">
-        <color rgba="0.75 0.75 0.75 1"/>
+      <material name="black">
+        <color rgba="0.1 0.1 0.1 1"/>
       </material>
     </visual>
